File: EurorackPSU.sch (KiCad schematic (older format))
At the start: 44 parts, among them J1 Conn_01x02, J2 Conn_01x03_Male, J3 Conn_01x03, J4 Conn_01x03_Male, U1 lt8638s, U2 lt8638s

Commit message: Assigned connectors for power input and output, and exported the netlist again
Parts:
- J1: footprint (none) -> Connector_Molex:Molex_Mini-Fit_Sr_42819-22XX_1x02_P10.00mm_Vertical
- J3: footprint (none) -> Connector_Molex:Molex_Mini-Fit_Sr_42819-32XX_1x03_P10.00mm_Vertical
Changed lines of the file:
@@
 F 0 "J3" H 11130 3992 50  0000 L CNN
 F 1 "Conn_01x03" H 11130 3901 50  0000 L CNN
-F 2 "" H 11050 3950 50  0001 C CNN
+F 2 "Connector_Molex:Molex_Mini-Fit_Sr_42819-32XX_1x03_P10.00mm_Vertical" H 11050 3950 50  0001 C CNN
 F 3 "~" H 11050 3950 50  0001 C CNN
 	1    11050 3950
@@
 F 0 "J1" H 668 1167 50  0000 C CNN
 F 1 "Conn_01x02" H 668 1076 50  0000 C CNN
-F 2 "" H 750 950 50  0001 C CNN
+F 2 "Connector_Molex:Molex_Mini-Fit_Sr_42819-22XX_1x02_P10.00mm_Vertical" H 750 950 50  0001 C CNN
 F 3 "~" H 750 950 50  0001 C CNN
 	1    750  950

Commit message: Added net name for power input, added more vias, and more
Connections:
- net +VDC: now reaches C1.1, C12.1, C13.1, C14.1, C15.1, C2.1, C3.1, C4.1, J1.1 (Pin_1), J2.1 (Pin_1), J4.1 (Pin_1), R1.1, R8.1, U1.15 (Vin), U1.16 (Vin), U1.17 (Vin), U1.18 (Vin), U2.15 (Vin), U2.16 (Vin), U2.17 (Vin), U2.18 (Vin)
Changed lines of the file:
@@
 Wire Wire Line
 	10750 1700 10750 3850
+$Comp
+L power:+VDC #PWR?
+U 1 1 60C9456F
+P 1400 800
+F 0 "#PWR?" H 1400 700 50  0001 C CNN
+F 1 "+VDC" H 1400 1075 50  0000 C CNN
+F 2 "" H 1400 800 50  0001 C CNN
+F 3 "" H 1400 800 50  0001 C CNN
+	1    1400 800
+	1    0    0    -1
+$EndComp
+Wire Wire Line
+	1400 800  1400 950
 $EndSCHEMATC
